File: Boards/Analog_Board/AnalogBoard_Rev0/Tremolo.sch (KiCad schematic (older format))
At the start: 30 parts

Commit message: analog board done awhile ago lol
Parts:
- added 9V, GND1, GND2, GND? (x2), PWR_IN: Wirepad, Connector_Wire:SolderWirePad_1x01_Drill1mm, symbol Pinebox:Wirepad
- added C1, C2: 100uF, Capacitor_THT:CP_Radial_D5.0mm_P2.00mm, symbol Device:CP
- added C5: 100uF, Capacitor_THT:CP_Radial_D6.3mm_P2.50mm, symbol Device:CP
- added C?: 4.7u, symbol Device:C
- added C?: 47u, symbol Device:C
- added D? (x2): 1N914, Diode_THT:D_DO-35_SOD27_P7.62mm_Horizontal, symbol Device:D
- added D?: B120-E3, Diode_SMD:D_SMA, symbol Diode:B120-E3
- added D?: D_Zener, symbol Device:D_Zener
- added D?: 10.2, symbol Device:D_Zener
- added J? (x3): AudioJack3_Switch, symbol Connector:AudioJack3_Switch
- added J?: AudioJack3_Switch, Pinebox:Jack_0.25in_TRS_Switched, symbol Connector:AudioJack3_Switch
- added J? (x2): Conn_01x02_Male, symbol Connector:Conn_01x02_Male
- added K?: RT42xxxx, Relay_THT:Relay_DPDT_Schrack-RT2-FormC_RM5mm, symbol Relay:RT42xxxx
- added Q?: MMBT3904, Package_TO_SOT_SMD:SOT-23, symbol Transistor_BJT:MMBT3904
- added Q?: Q_PMOS_DGS, symbol Device:Q_PMOS_DGS
- added R?: 100k, symbol Device:R
- added R?: 3.3k, symbol Device:R
- added R?: 10k, symbol Device:R
- added R?: 47k, symbol Device:R
- added R?: 1k, symbol Device:R
- added U1: LTC1044, Package_SO:SO-8_3.9x4.9mm_P1.27mm, symbol Regulator_SwitchedCapacitor:LTC1044
- added U? (x2): TLP222A-2, Package_DIP:DIP-8_W7.62mm, symbol Relay_SolidState:TLP222A-2
- added U? (x3): OPA2134, symbol Amplifier_Operational:OPA2134
Connections:
- net labels added: ENV_OUT, MUTE2, PWR_IN, RLY_SET, SW_STREO_1, SW_STREO_2
- wire segments 108 -> 216
- no-connect marks 0 -> 2
Other:
- note added: "Reverse & Overvoltage Protection"
- moved on the sheet: C?, R?, RV?, U?A, U?B, U?C
