File: Boards/Analog_Board/AnalogBoard_Rev0/_autosave-Tremolo.sch (KiCad schematic (older format))
At the start: 50 parts, among them U1 LTC1044

Commit message: analog board done awhile ago lol
Parts:
- removed D2: 1N4001, Diode_THT:D_DO-41_SOD81_P10.16mm_Horizontal, symbol Diode:1N4001
- added 9V, PWR_IN: Wirepad, Connector_Wire:SolderWirePad_1x01_Drill1mm, symbol Pinebox:Wirepad
- added C?: 4.7u, symbol Device:C
- added C?: 47u, symbol Device:C
- added D? (x2): 1N914, Diode_THT:D_DO-35_SOD27_P7.62mm_Horizontal, symbol Device:D
- added D?: D_Zener, symbol Device:D_Zener
- added D?: 10.2, symbol Device:D_Zener
- added Q?: Q_PMOS_DGS, symbol Device:Q_PMOS_DGS
- added R?: 100k, symbol Device:R
- added R?: 3.3k, symbol Device:R
- added R?: 10k, symbol Device:R
- added R?: 47k, symbol Device:R
- added R?: 1k, symbol Device:R
- added U? (x3): OPA2134, symbol Amplifier_Operational:OPA2134
- J?: footprint (none) -> Pinebox:Jack_0.25in_TRS_Switched
Connections:
- net labels added: ENV_OUT, PWR_IN, SW_STREO_1, SW_STREO_2
- net labels removed: SW_STREO, SW_STREO_IN
- wire segments 174 -> 216
Other:
- note added: "Reverse & Overvoltage Protection"
- moved on the sheet: C1, C2, C5, U?C
