File: Boards/Analog_Board/AnalogBoard_Rev0/AnalogBoard_Rev0.sch (KiCad schematic (older format))
At the start: 0 parts

Commit message: analog board done awhile ago lol
Parts:
- added C1, C2: 47n, Capacitor_THT:C_Rect_L7.2mm_W4.5mm_P5.00mm_FKS2_FKP2_MKS2_MKP2, symbol Device:C
- added C10: 4.7u, Capacitor_THT:CP_Radial_D5.0mm_P2.00mm, symbol Device:C
- added C11: 47u, Capacitor_THT:CP_Radial_D5.0mm_P2.00mm, symbol Device:C
- added C12, C13: 470n, Capacitor_THT:C_Rect_L7.2mm_W4.5mm_P5.00mm_FKS2_FKP2_MKS2_MKP2, symbol Device:C
- added C14, C15, C16, C17, C18, C19, C20, C21, C22, C23: 100n, Capacitor_SMD:C_0603_1608Metric_Pad1.05x0.95mm_HandSolder, symbol MF_Passives:CAPACITOR_NP_0603
- added C3, C6, C9: 100uF, Capacitor_THT:CP_Radial_D5.0mm_P2.00mm, symbol Device:CP
- added C4, C5, C7, C8: 1n, Capacitor_THT:C_Rect_L7.2mm_W4.5mm_P5.00mm_FKS2_FKP2_MKS2_MKP2, symbol Device:C
- added D1: 10.2, Diode_THT:D_DO-35_SOD27_P7.62mm_Horizontal, symbol Device:D_Zener
- added D2, D3: 1N914, Diode_THT:D_DO-35_SOD27_P7.62mm_Horizontal, symbol Device:D
- added D4: D_Zener, Diode_THT:D_DO-34_SOD68_P7.62mm_Horizontal, symbol Device:D_Zener
- added D5: B120-E3, Diode_THT:D_DO-35_SOD27_P7.62mm_Horizontal, symbol Diode:B120-E3
- added H1, H2, H3, H4: MountingHole, MountingHole:MountingHole_3.2mm_M3, symbol Mechanical:MountingHole
- added J1, J2, J5, J6: AudioJack3_Switch, Pinebox:Jack_0.25in_TRS_Switched, symbol Connector:AudioJack3_Switch
- added J10, J11, J12, J13, J14, J7, J8, J9: Conn_01x02_Female, Connector_PinSocket_2.54mm:PinSocket_1x02_P2.54mm_Vertical, symbol Connector:Conn_01x02_Female
- added J15, J16, J17, J18, J19, J20, J21, J22, J24, J26, J27, J29, J3, J30, J31, J4: Conn_01x02_Male, Connector_PinHeader_2.54mm:PinHeader_1x02_P2.54mm_Vertical, symbol Connector:Conn_01x02_Male
- added J23, J25: Conn_01x03_Male, Connector_PinHeader_2.54mm:PinHeader_1x03_P2.54mm_Vertical, symbol Connector:Conn_01x03_Male
- added J28: Barrel_Jack_MountingPin, Connector_BarrelJack:BarrelJack_CUI_PJ-063AH_Horizontal_CircularHoles, symbol Connector:Barrel_Jack_MountingPin
- added JP1, JP2: JMP_NC, Jumper:SolderJumper-2_P1.3mm_Bridged_Pad1.0x1.5mm, symbol Jumper:Jumper_2_Bridged
- added K1: IM05, Pinebox:Relay_DPDT_NL_TE_IM05GR, symbol Relay:IM05
- added Q1: Q_PMOS_DGS, Package_TO_SOT_THT:TO-92L_Inline, symbol Device:Q_PMOS_DGS
- added Q2: MMBT3904, Package_TO_SOT_SMD:SOT-23, symbol Transistor_BJT:MMBT3904
- added R1, R2: 1M, Resistor_THT:R_Axial_DIN0207_L6.3mm_D2.5mm_P7.62mm_Horizontal, symbol Device:R
- added R10: 47k, Resistor_THT:R_Axial_DIN0207_L6.3mm_D2.5mm_P7.62mm_Horizontal, symbol Device:R
- added R11, R12, R13: 1k, Resistor_THT:R_Axial_DIN0207_L6.3mm_D2.5mm_P7.62mm_Horizontal, symbol Device:R
- added R14: 4.7k, Resistor_THT:R_Axial_DIN0207_L6.3mm_D2.5mm_P7.62mm_Horizontal, symbol Device:R
- added R15, R16: 630, Resistor_THT:R_Axial_DIN0207_L6.3mm_D2.5mm_P7.62mm_Horizontal, symbol Device:R
- added R3, R4, R6, R7: 470k, Resistor_THT:R_Axial_DIN0207_L6.3mm_D2.5mm_P7.62mm_Horizontal, symbol Device:R
- added R5: 3.3k, Resistor_THT:R_Axial_DIN0207_L6.3mm_D2.5mm_P7.62mm_Horizontal, symbol Device:R
- added R8: 100k, Resistor_THT:R_Axial_DIN0207_L6.3mm_D2.5mm_P7.62mm_Horizontal, symbol Device:R
- added R9: 10k, Resistor_THT:R_Axial_DIN0207_L6.3mm_D2.5mm_P7.62mm_Horizontal, symbol Device:R
- added RV1, RV2, RV3, RV4: 50k, Potentiometer_THT:Potentiometer_Bourns_3386F_Vertical, symbol Device:R_POT_TRIM_US
- added U1, U2, U3, U4, U5: OPA2134, Package_DIP:DIP-8_W7.62mm, symbol Amplifier_Operational:OPA2134
- added U10: TLP222A-2, Package_DIP:DIP-8_W7.62mm, symbol Relay_SolidState:TLP222A-2
- added U11, U12, U13, U7, U8, U9: NSL-32, Pinebox:Luna_NSL-32_Vertical, symbol Isolator:NSL-32
- added U6: TC7662Bx0A, Package_SO:SOIC-8_3.9x4.9mm_P1.27mm, symbol Converter_DCDC:TC7662Bx0A
Connections:
- new net: C4.2, J7.2 (Pin_2), J8.2 (Pin_2), K1.2, R3.1, U1.1, U1.2 (-), U5.3 (+)
- new net: C1.1, R1.2, U1.3 (+)
- new net: C7.2, J13.1 (Pin_1), J7.1 (Pin_1), R3.2, U3.3 (+)
- new net: C5.2, J10.2 (Pin_2), J9.2 (Pin_2), K1.7, R4.1, U2.1, U2.2 (-)
- new net: C2.1, R2.2, U2.3 (+)
- new net: C4.1, J11.1 (Pin_1), J8.1 (Pin_1), R6.2, U3.5 (+)
- new net: K1.4, R12.2, U1.7
- new net: R12.1, RV1.3, U12.3 (R)
- new net: C12.1, J3.2 (Pin_2), RV3.1, U10.8
- new net: C12.2, K1.3
- new net: C8.2, J14.1 (Pin_1), J9.1 (Pin_1), R4.2, U4.3 (+)
- new net: C5.1, J10.1 (Pin_1), J12.1 (Pin_1), R7.2, U4.5 (+)
- new net: K1.5, R13.2, U2.7
- new net: C13.1, J4.2 (Pin_2), RV4.1, U10.6
- new net: C13.2, K1.6
- new net: R13.1, RV2.3, U13.3 (R)
- new net: C6.1, U6.2 (CAP+)
- new net: C6.2, U6.4 (CAP-)
- new net: R15.2, U10.1
- new net: R16.2, U10.3
- new net: Q2.1 (B), R14.2
- new net: JP2.2 (B), Q2.2 (E)
- new net: D5.2 (A), K1.8, Q2.3 (C)
- new net: D5.1 (K), JP1.1 (A), K1.1
- new net: D2.1 (K), D3.2 (A), U5.1
- new net: D2.2 (A), R5.1, R8.1, U5.2 (-)
- new net: D3.1 (K), R8.2, R9.1
- new net: C10.2, R10.1, R9.2, U5.5 (+)
- new net: R11.1, U5.6 (-), U5.7
- new net: J17.1 (Pin_1), U9.1 (A)
- new net: J17.2 (Pin_2), U9.2 (K)
- new net: J18.1 (Pin_1), U11.1 (A)
- new net: J18.2 (Pin_2), U11.2 (K)
- new net: J16.1 (Pin_1), U8.1 (A)
- new net: J16.2 (Pin_2), U8.2 (K)
- new net: J15.1 (Pin_1), U7.1 (A)
- new net: J15.2 (Pin_2), U7.2 (K)
- new net: J21.1 (Pin_1), U12.1 (A)
- new net: J21.2 (Pin_2), U12.2 (K)
- new net: J22.1 (Pin_1), U13.1 (A)
- new net: J22.2 (Pin_2), U13.2 (K)
- new net +9V: C14.2, C16.2, C18.2, C20.2, C22.2, C3.1, D1.1 (K), J24.2 (Pin_2), J25.3 (Pin_3), JP1.2 (B), Q1.3 (S), U1.8 (V+), U2.8 (V+), U3.8 (V+), U4.8 (V+), U5.8 (V+), U6.1 (BOOST), U6.8 (V+)
- new net -9V: C15.1, C17.1, C19.1, C21.1, C23.1, C9.2, J25.2 (Pin_2), U1.4 (V-), U2.4 (V-), U3.4 (V-), U4.4 (V-), U5.4 (V-), U6.5 (VOUT)
- new net ENV_OUT: C11.2, D4.1 (K), R11.2
- new net GND: C10.1, C11.1, C14.1, C15.2, C16.1, C17.2, C18.1, C19.2, C20.1, C21.2, C22.1, C23.2, C3.2, C7.1, C8.1, C9.1, D1.2 (A), D4.2 (A), J11.2 (Pin_2), J12.2 (Pin_2), J13.2 (Pin_2), J14.2 (Pin_2), J24.1 (Pin_1), J25.1 (Pin_1), J28.1, J28.MP (MountPin), J29.1 (Pin_1), J3.1 (Pin_1), J31.1 (Pin_1), J4.1 (Pin_1), JP2.1 (A), Q1.2 (G), R1.1, R10.2, R2.1, R5.2, R6.1, R7.1, RV3.3, RV4.3, U1.5 (+), U10.5, U10.7, U2.5 (+), U6.3 (GND)
- new net GNDD: J23.1 (Pin_1), U10.2, U10.4
- new net IN1: C1.2, J1.T, J2.TN
- new net IN2: C2.2, J2.T
- new net LDRA_1: J19.2 (Pin_2), U3.1, U3.2 (-), U7.4 (R)
- new net LDRA_2: J19.1 (Pin_1), J20.1 (Pin_1), RV1.1, RV1.2, U1.6 (-), U12.4 (R), U7.3 (R), U8.3 (R)
- new net LDRB_1: J20.2 (Pin_2), U3.6 (-), U3.7, U8.4 (R)
- new net LDRC_1: J26.2 (Pin_2), U4.1, U4.2 (-), U9.4 (R)
- new net LDRC_2: J26.1 (Pin_1), J27.1 (Pin_1), RV2.1, RV2.2, U11.3 (R), U13.4 (R), U2.6 (-), U9.3 (R)
- new net LDRD_1: J27.2 (Pin_2), U11.4 (R), U4.6 (-), U4.7
- new net MUTE1: J23.3 (Pin_3), R15.1
- new net MUTE2: J23.2 (Pin_2), R16.1
- new net OUT1: J5.T, RV3.2
- new net OUT2: J6.T, RV4.2
- new net PWR_IN: J28.2, J29.2 (Pin_2), Q1.1 (D)
- new net RLY_SET: J31.2 (Pin_2), R14.1
- new net SW_STREO_1: J1.SN, J30.1 (Pin_1)
- new net SW_STREO_2: J2.SN, J30.2 (Pin_2)
- no-connect marks 0 -> 19
Other:
- note added: "Add volume opto driver stage"
- note added: "Reverse & Overvoltage Protection"
- note added: "To Digital Board"

Commit message: r2 boards released, finally pushing
Parts:
- C14, C15, C16, C17, C18, C19, C20, C21, C22, C23: symbol MF_Passives:CAPACITOR_NP_0603 -> AnalogBoard_Rev0-rescue:CAPACITOR_NP_0603-MF_Passives
- U6: symbol Converter_DCDC:TC7662Bx0A -> AnalogBoard_Rev0-rescue:TC7662Bx0A-Converter_DCDC
Changed lines of the file:
@@
 	6650 1050 6650 1150
 $Comp
-L Converter_DCDC:TC7662Bx0A U6
+L AnalogBoard_Rev0-rescue:TC7662Bx0A-Converter_DCDC U6
 U 1 1 6173B633
 P 5200 1900
@@
 $EndComp
 $Comp
-L MF_Passives:CAPACITOR_NP_0603 C14
+L AnalogBoard_Rev0-rescue:CAPACITOR_NP_0603-MF_Passives C14
 U 1 1 61F0FF0B
 P 7150 1700
@@
 	7150 1900 7150 1800
 $Comp
-L MF_Passives:CAPACITOR_NP_0603 C15
+L AnalogBoard_Rev0-rescue:CAPACITOR_NP_0603-MF_Passives C15
 U 1 1 6218B379
 P 7150 2100
@@
 Connection ~ 7150 1900
 $Comp
-L MF_Passives:CAPACITOR_NP_0603 C16
+L AnalogBoard_Rev0-rescue:CAPACITOR_NP_0603-MF_Passives C16
 U 1 1 622A5ECF
 P 8150 1700
@@
 	8150 1900 8150 1800
 $Comp
-L MF_Passives:CAPACITOR_NP_0603 C17
+L AnalogBoard_Rev0-rescue:CAPACITOR_NP_0603-MF_Passives C17
 U 1 1 622A5EE6
 P 8150 2100
@@
 Connection ~ 8350 2200
 $Comp
-L MF_Passives:CAPACITOR_NP_0603 C18
+L AnalogBoard_Rev0-rescue:CAPACITOR_NP_0603-MF_Passives C18
 U 1 1 622D8B8A
 P 9100 1700
@@
 	9100 1900 9100 1800
 $Comp
-L MF_Passives:CAPACITOR_NP_0603 C19
+L AnalogBoard_Rev0-rescue:CAPACITOR_NP_0603-MF_Passives C19
 U 1 1 622D8BA1
 P 9100 2100
@@
 Connection ~ 9300 2200
 $Comp
-L MF_Passives:CAPACITOR_NP_0603 C20
+L AnalogBoard_Rev0-rescue:CAPACITOR_NP_0603-MF_Passives C20
 U 1 1 623220CB
 P 10100 1700
@@
 	10100 1900 10100 1800
 $Comp
-L MF_Passives:CAPACITOR_NP_0603 C21
+L AnalogBoard_Rev0-rescue:CAPACITOR_NP_0603-MF_Passives C21
 U 1 1 623220E2
 P 10100 2100
@@
 Connection ~ 10300 2200
 $Comp
-L MF_Passives:CAPACITOR_NP_0603 C22
+L AnalogBoard_Rev0-rescue:CAPACITOR_NP_0603-MF_Passives C22
 U 1 1 62358DE8
 P 11100 1700
@@
 	11100 1900 11100 1800
 $Comp
-L MF_Passives:CAPACITOR_NP_0603 C23
+L AnalogBoard_Rev0-rescue:CAPACITOR_NP_0603-MF_Passives C23
 U 1 1 62358DFF
 P 11100 2100
