File: Boards/Analog Board Rev 2/AnalogBoard_Rev2/AnalogBoard_Rev2.sch (KiCad schematic (older format))
At the start: 56 parts, among them J1 Conn_01x06_Male, J2 Conn_01x10_Male, J3 Conn_01x06_Male, J4 Conn_01x08_Male, SW1 SW_DIP_x04, U1 OPA2134, U12 NSL-32, U13 NSL-32, U2 OPA2134, U3 OPA2134, U4 OPA2134, U5 OPA2134, U6 NSL-32, U7 NSL-32, U8 NSL-32, U9 NSL-32

Commit message: reorg pt 1
Reorganizing, deleted a bunch of stuff. Probably will reorg some more
Parts:
- RV1, RV2, RV3, RV4: symbol Device:R_POT_TRIM_US -> AnalogBoard_Rev2-rescue:R_POT_TRIM_US-Device
