File: Boards/Digital Board Rev 2/Digital Board Rev 2/Digital Board Rev 2.kicad_pcb (KiCad board)
At the start: 4 copper layers, 59.5 x 96.3 mm, 91 parts, among them J1 Conn_01x02_Male, J10 AudioJack3_Switch, J11 Conn_01x10_Female, J12 Barrel_Jack, J13 Conn_01x06_Female, J14 Conn_01x06_Female, J15 Conn_01x03_Male, J2 Conn_01x02_Male, J3 Conn_01x06_Male, J4 Conn_01x08_Female, J5 AudioJack3_Switch, J6 AudioJack3_Switch, J7 AudioJack3_Switch, J8 AudioJack3_Switch, J9 AudioJack3_Switch, K1 IM05, Q1 BSS83P, Q25 MMBT3904, SW1 SW_SPDT_MSM, SW2 SW_SPDT_MSM, SW3 SW_SPDT_MSM, U1 STM32F303R6Tx, U26 TLP222A-2, U27 NCP1117-3.3_SOT223, U28 TC7662Bx0A, Y1 8MHz

Commit message: reorg pt 1
Reorganizing, deleted a bunch of stuff. Probably will reorg some more
Other:
- net class Default removed
