File: Boards/Digital Board Rev 2/Digital Board Rev 2/Digital Board Rev 2.sch (KiCad schematic (older format))
At the start: 34 parts, among them J1 Conn_01x02_Male, J11 Conn_01x10_Female, J13 Conn_01x06_Female, J14 Conn_01x06_Female, J15 Conn_01x03_Male, J2 Conn_01x02_Male, J3 Conn_01x06_Male, J4 Conn_01x08_Female, U1 STM32F303R6Tx, Y1 8MHz

Commit message: reorg pt 1
Reorganizing, deleted a bunch of stuff. Probably will reorg some more
Parts:
- JP1: symbol Device:Jumper -> Digital-Board-Rev-2-rescue:Jumper-Device
- NT1, NT2, NT3, NT4: symbol Device:Net-Tie_2 -> Digital-Board-Rev-2-rescue:Net-Tie_2-Device
