File: Rev_1/Digital_Board_Rev_1/Digital_Board_Rev_1.kicad_pcb (KiCad board)
At the start: 4 copper layers, 101.6 x 101.6 mm, 135 parts, among them J1 USB_MICRO_RIGHT, J13 CON_01X02_PTH_2.54MM, J14 CON_01X04_PTH_2.54MM, J17 CON_01X02_PTH_2.54MM, J20 AudioJack3_Switch, J21 Barrel_Jack, J22 CON_01X02_PTH_2.54MM, J6 Conn_01x02_Male, J7 Conn_01x02_Male, J8 Conn_01x02_Male, J9 Conn_01x02_Male, SW1 CON_01X02_PTH_2.54MM, SW1 SW_DIP_x04, SW2 CON_01X02_PTH_2.54MM, SW2 SW_DIP_x02, U1 FT230XS-R, U10 NPN_BJTMMBT3904_SOT-23-3, U11 NSL-32, U12 NSL-32, U13 STM32F030RCTx, U14 CPC1017N, U15 CPC1017N, U2 NCP1117LPST33T3G, U3 MCP42050, U4 MCP42050, U5 NPN_BJTMMBT3904_SOT-23-3, U6 NPN_BJTMMBT3904_SOT-23-3, U7 NSL-32, U8 NSL-32, U9 NPN_BJTMMBT3904_SOT-23-3

Commit message: Pivoting to Passive Jack Boards
Finalized layout for input/output Jack Boards, which are now completely passive and connected with board-to-board connectors. Schematics are not updated yet, just figuring out placement/dimensions.
Other:
- net class Default removed
