File: Rev_3/Digital_Board_Rev_3/Analog.kicad_sch (KiCad schematic)
At the start: 52 parts, among them U10 OPA1688IDR, U11 OPA1688IDR, U12 OPA1688IDR, U13 OPA1688IDR, U8 TLE2426xD, U9 OPA1688IDR

Commit message: Backing up before windows crash debug
Parts:
- removed C21: 100u, Capacitor_SMD:CP_Elec_8x6.2, symbol #gplm:cap/CAP-3005-100U
- removed C22, C24: 22n, Capacitor_THT:C_Rect_L7.2mm_W3.0mm_P5.00mm_FKS2_FKP2_MKS2_MKP2, symbol #gplm:cap/CAP-1002-0003
- removed C23: 10u, Capacitor_SMD:C_1206_3216Metric, symbol #gplm:cap/CAP-4006-010U
- removed C25, C33: 1u, Capacitor_SMD:C_0603_1608Metric, symbol #gplm:cap/CAP-4004-001U
- removed C26, C27: 22p, Capacitor_SMD:C_0402_1005Metric, symbol #gplm:cap/CAP-4001-022P
- removed C30, C32, C36, C37, C40, C41, C42, C43, C44, C45: 100n, Capacitor_SMD:C_0402_1005Metric, symbol #gplm:cap/RES-4003-100N
- removed C31: 10u, Capacitor_SMD:CP_Elec_6.3x5.8, symbol #gplm:cap/CAP-3005-010U
- removed C34, C35, C38, C39: 10n, Capacitor_THT:C_Rect_L7.2mm_W3.0mm_P5.00mm_FKS2_FKP2_MKS2_MKP2, symbol #gplm:cap/CAP-1002-0001
- removed OP1, OP2, OP3, OP4, OP5, OP6: NSL-32, g-opt:Luna_NSL-32_Vertical, symbol #gplm:opt/OPT-0002-0001
- removed R20: 1, Resistor_SMD:R_0603_1608Metric, symbol #gplm:res/RES-2001-001R
- removed R21, R22, R23, R24: 1M, Resistor_SMD:R_0603_1608Metric, symbol #gplm:res/RES-2001-001M
- removed R25, R26: 100k, Resistor_SMD:R_0603_1608Metric, symbol #gplm:res/RES-2001-100K
- removed R27, R28, R29, R30: 39k, Resistor_SMD:R_0603_1608Metric, symbol #gplm:res/RES-2001-039K
- removed R31, R32: 100, Resistor_SMD:R_0603_1608Metric, symbol #gplm:res/RES-2001-100R
- removed R33, R34: 330, Resistor_SMD:R_0603_1608Metric, symbol #gplm:res/RES-2001-330R
- removed RV5, RV6: B1k, g-pot:Potentiometer_Bourns_3214G_Horizontal, symbol #gplm:pot/POT-0008-B102
- removed U10, U11, U12, U13, U9: OPA1688IDR, Package_SO:SOIC-8_3.9x4.9mm_P1.27mm, symbol #gplm:ana/ANA-1001-2000
- removed U8: TLE2426xD, Package_SO:SOIC-8_3.9x4.9mm_P1.27mm, symbol Reference_Voltage:TLE2426xD
Other:
- note removed: "408 Hz"
- note removed: "Coupling caps on Output Board"
- note removed: "Gives gain of ~1 at 100% duty"
- note removed: "OPA1679?"
- note removed: "Trimpot just for testing. Install either pot or R22."
