File: Rev_3/Digital_Board_Rev_3/Digital_Board_Rev3.kicad_pcb (KiCad board)
At the start: 4 copper layers, 59 x 93 mm, 79 parts, among them K1 IM05GR, Q1 MMBT3904, Q2 DMP3099L, SW2 SW_SPDT_MSM, U1 TPSM84338RCJR, U2 STM32G474VBTx, U3 ADP7142ARDZ, U4 TLP2361, U5 OPA2134, U6 TLP170AM, U7 TLP170AM

Commit message: Backing up before windows crash debug
Parts:
- moved U2 1.35 mm to (96.5, 121.0)
Changed lines of the file:
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@@
 		(39 "User.1" user "Enclosure")
 		(41 "User.2" user "Offboard.Objects")
-		(45 "User.4" user "Other.PCBs")
+		(43 "User.3" user "Labels")
+		(45 "User.4" user "PCB.DigitalBoard")
+		(47 "User.5" user "PCB.OutputBoard")
 	)
 	(setup
@@
 		(allow_soldermask_bridges_in_footprints no)
 		(tenting front back)
-		(grid_origin 80 50)
+		(grid_origin 100 50)
 		(pcbplotparams
 			(layerselection 0x00000000_00000000_55555555_5755f5ff)
-			(plot_on_all_layers_selection 0x00000000_00000000_00000000_02000000)
+			(plot_on_all_layers_selection 0x00000000_00000000_00000000_00000000)
 			(disableapertmacros no)
 			(usegerberextensions no)
@@
 			(dashed_line_dash_ratio 12.000000)
 			(dashed_line_gap_ratio 3.000000)
-			(svgprecision 6)
+			(svgprecision 4)
 			(plotframeref no)
 			(mode 1)
@@
 			(psa4output no)
 			(plot_black_and_white yes)
-			(plotinvisibletext no)
 			(sketchpadsonfab no)
 			(plotpadnumbers no)
@@
 			(outputformat 1)
 			(mirror no)
-			(drillshape 0)
+			(drillshape 1)
 			(scaleselection 1)
 			(outputdirectory "")
@@
 	(footprint "Package_QFP:LQFP-100_14x14mm_P0.5mm"
 		(layer "B.Cu")
-		(at 95.175 120.75)
+		(at 96.5 121)
 		(descr "LQFP, 100 Pin (https://www.nxp.com/docs/en/package-information/SOT407-1.pdf), generated with kicad-footprint-generator ipc_gullwing_generator.py")
 		(tags "LQFP QFP")
